Commit message: fixes to get rviz showing laser scan values

File: urdf/gazebo_tags/gazebo_plugins.xacro (robot description, xacro)
@@ -10,6 +10,6 @@
             <wheel_separation>0.215</wheel_separation>
             <wheel_radius>0.06</wheel_radius>
-            <frame_id>odom</frame_id>
-            <child_frame_id>base_footprint</child_frame_id>
+            <frame_id>camlidarbot/odom</frame_id> <!--Best to use prefixes ('camlidarbot' for example) and to set the prefix on the RVIZ config too-->
+            <child_frame_id>camlidarbot/base_footprint</child_frame_id> <!--Best to use prefixes ('camlidarbot' for example) and to set the prefix on the RVIZ config too-->
             <!--<topic>cmd_vel</topic> -->
         </plugin>
@@ -23,3 +23,45 @@
         </plugin>
     </gazebo>
+    <!-- IF USING SENSORS MUST INCLUDE THE BELOW -->
+    <gazebo>
+        <plugin filename="gz-sim-sensors-system" name="gz::sim::systems::Sensors">
+            <render_engine>ogre2</render_engine>
+        </plugin>
+    </gazebo>
+    <!--=========================================-->
+    <gazebo reference="lidar_link">
+        <sensor name='gpu_lidar' type='gpu_lidar'>"
+            <pose relative_to='lidar_link'>0 0 0 0 0 0</pose>
+            <topic>scan</topic>
+            <update_rate>2</update_rate>
+            <always_on>1</always_on>
+            <visualize>1</visualize>
+            <lidar>
+                <scan>
+                    <horizontal>
+                        <samples>640</samples>
+                        <resolution>1</resolution>
+                        <min_angle>-1.396263</min_angle>
+                        <max_angle>1.396263</max_angle>
+                    </horizontal>
+                    <!--<vertical> Not needed if not scanning vertically
+                        <samples>1</samples>
+                        <resolution>0.01</resolution>
+                        <min_angle>0</min_angle>
+                        <max_angle>0</max_angle>
+                    </vertical>-->
+                </scan>
+                <range>
+                    <min>0.08</min>
+                    <max>10.0</max>
+                    <resolution>0.01</resolution>
+                </range>
+                <noise>
+                    <type>gaussian</type>
+                    <mean>0.0</mean>
+                    <stddev>0.001</stddev>
+                </noise>
+            </lidar>
+        </sensor>
+    </gazebo>
 </robot>

File: urdf/modules/camlidarbot.xacro (robot description, xacro)
@@ -3,4 +3,18 @@
 <!-- Onshape document_id a4ea59dba35f5caeb271cde4 -->
 <robot xmlns:xacro="http://www.ros.org/wiki/xacro">
+  <!-- Joint map -->
+  <!--<link name="map"/>
+  <joint name="map_joint" type="static">
+      <parent link="map" />
+      <child link="odom" />
+      <origin xyz="0 0 0" rpy="0 0 0" />
+  </joint>-->
+  <!-- Joint odom -->
+  <!--<link name="odom"/>
+  <joint name="odom_joint" type="static">
+      <parent link="odom" />
+      <child link="base_footprint" />
+      <origin xyz="0 0 0" rpy="0 0 0" />
+  </joint>-->
   <!-- Link base footprint -->
   <link name="base_footprint"/>
@@ -65,35 +79,4 @@
     <child link="lidar_link"/>
   </joint>
-  <frame name="lidar_frame" attached_to='lidar_link'>
-    <pose>0.8 0 0.5 0 0 0</pose>
-  </frame>
-  <sensor name='gpu_lidar' type='gpu_lidar'>"
-    <pose relative_to='lidar_frame'>0 0 0 0 0 0</pose>
-    <topic>lidar</topic>
-    <update_rate>10</update_rate>
-    <ray>
-        <scan>
-            <horizontal>
-                <samples>640</samples>
-                <resolution>1</resolution>
-                <min_angle>-1.396263</min_angle>
-                <max_angle>1.396263</max_angle>
-            </horizontal>
-            <vertical>
-                <samples>1</samples>
-                <resolution>0.01</resolution>
-                <min_angle>0</min_angle>
-                <max_angle>0</max_angle>
-            </vertical>
-        </scan>
-        <range>
-            <min>0.08</min>
-            <max>10.0</max>
-            <resolution>0.01</resolution>
-        </range>
-    </ray>
-    <always_on>1</always_on>
-    <visualize>true</visualize>
-  </sensor>
   <!-- Link camera -->
   <link name="camera_link">

Commit message: gazebo camera plugin setup and urdf folder structure improvements

File: urdf/gazebo_tags/gazebo_plugins.xacro (robot description, xacro)
@@ -2,4 +2,5 @@
 <!--AS WE HAVE FOUR WHEELED ROBOT, WE WILL DEFINE TWO LEFT JOINTS AND TWO RIGHT JOINTS-->
 <robot xmlns:xacro="http://www.ros.org/wiki/xacro">
+<!-- =============== DiffDrive =============== -->
     <gazebo>
         <plugin filename="gz-sim-diff-drive-system" name="gz::sim::systems::DiffDrive">
@@ -23,5 +24,6 @@
         </plugin>
     </gazebo>
-    <!-- IF USING SENSORS MUST INCLUDE THE BELOW -->
+<!--=========================================-->
+<!-- IF USING SENSORS MUST INCLUDE THE BELOW -->
     <gazebo>
         <plugin filename="gz-sim-sensors-system" name="gz::sim::systems::Sensors">
@@ -29,5 +31,5 @@
         </plugin>
     </gazebo>
-    <!--=========================================-->
+<!-- =========== Lidar Sensor ============ -->
     <gazebo reference="lidar_link">
         <sensor name='gpu_lidar' type='gpu_lidar'>"
@@ -65,3 +67,33 @@
         </sensor>
     </gazebo>
+<!--=========================================-->
+<!-- =========== Camera Sensor ============ -->
+    <gazebo reference="camera_link">
+        <sensor name="camera" type="camera">
+            <camera>
+                <horizontal_fov>1.3962634</horizontal_fov>
+                <image>
+                    <width>640</width>
+                    <height>480</height>
+                    <format>R8G8B8</format>
+                </image>
+                <clip>
+                    <near>0.1</near>
+                    <far>15</far>
+                </clip>
+                <noise>
+                    <type>gaussian</type>
+                    <mean>0.0</mean>
+                    <stddev>0.007</stddev>
+                </noise>
+                <optical_frame_id>camera_optical_link</optical_frame_id>
+                <camera_info_topic>camera/camera_info</camera_info_topic>
+            </camera>
+            <always_on>1</always_on>
+            <update_rate>20</update_rate>
+            <visualize>true</visualize>
+            <topic>camera/image_raw</topic>
+        </sensor>
+    </gazebo>
+<!--=========================================-->
 </robot>

File: urdf/modules/chassis_and_wheels.xacro (robot description, xacro)
@@ -3,18 +3,4 @@
 <!-- Onshape document_id a4ea59dba35f5caeb271cde4 -->
 <robot xmlns:xacro="http://www.ros.org/wiki/xacro">
-  <!-- Joint map -->
-  <!--<link name="map"/>
-  <joint name="map_joint" type="static">
-      <parent link="map" />
-      <child link="odom" />
-      <origin xyz="0 0 0" rpy="0 0 0" />
-  </joint>-->
-  <!-- Joint odom -->
-  <!--<link name="odom"/>
-  <joint name="odom_joint" type="static">
-      <parent link="odom" />
-      <child link="base_footprint" />
-      <origin xyz="0 0 0" rpy="0 0 0" />
-  </joint>-->
   <!-- Link base footprint -->
   <link name="base_footprint"/>
@@ -49,64 +35,4 @@
     </collision>
   </link>
-  <!-- Link lidar -->
-  <link name="lidar_link">
-    <inertial>
-      <origin xyz="-4.82929e-19 1.36409e-18 0.00735149" rpy="0 0 0"/>
-      <mass value="0.027159"/>
-      <inertia ixx="4.77113e-06" ixy="0" ixz="0" iyy="4.77113e-06" iyz="0" izz="8.40399e-06"/>
-    </inertial>
-    <!-- Part lidar -->
-    <visual>
-      <origin xyz="0 -1.53081e-19 0" rpy="0 -0 0"/>
-      <geometry>
-        <mesh filename="package://camlidarbot_description/assets/lidar.stl"/>
-      </geometry>
-      <material name="lidar_material">
-        <color rgba="0.301961 0.301961 0.301961 1"/>
-      </material>
-    </visual>
-    <collision>
-      <origin xyz="0 -1.53081e-19 0" rpy="0 -0 0"/>
-      <geometry>
-        <mesh filename="package://camlidarbot_description/assets/lidar.stl"/>
-      </geometry>
-    </collision>
-  </link>
-  <!-- Joint from chassis to lidar -->
-  <joint name="lidar_joint" type="fixed">
-    <origin xyz="-0.0440219 2.44392e-17 0.09" rpy="0 -0 0"/>
-    <parent link="chassis_link"/>
-    <child link="lidar_link"/>
-  </joint>
-  <!-- Link camera -->
-  <link name="camera_link">
-    <inertial>
-      <origin xyz="-5.3242e-19 -6.85029e-19 0.00414969" rpy="0 0 0"/>
-      <mass value="0.00103549"/>
-      <inertia ixx="3.58884e-08" ixy="0" ixz="0" iyy="4.57792e-08" iyz="0" izz="1.57304e-08"/>
-    </inertial>
-    <!-- Part camera -->
-    <visual>
-      <origin xyz="0 0 0" rpy="0 -0 0"/>
-      <geometry>
-        <mesh filename="package://camlidarbot_description/assets/camera.stl"/>
-      </geometry>
-      <material name="camera_material">
-        <color rgba="0.729412 0.25098 0.105882 1"/>
-      </material>
-    </visual>
-    <collision>
-      <origin xyz="0 0 0" rpy="0 -0 0"/>
-      <geometry>
-        <mesh filename="package://camlidarbot_description/assets/camera.stl"/>
-      </geometry>
-    </collision>
-  </link>
-  <!-- Joint from chassis to camera -->
-  <joint name="camera_joint" type="fixed">
-    <origin xyz="0.0811976 0 0.05" rpy="0 -0 1.5708"/>
-    <parent link="chassis_link"/>
-    <child link="camera_link"/>
-  </joint>
   <!-- Link rear_right_wheel -->
   <link name="rear_right_wheel_link">

File: urdf/robot.urdf.xacro (robot description, xacro)
@@ -1,5 +1,7 @@
 <?xml version="1.0" ?>
 <robot name="camlidarbot" xmlns:xacro="http://www.ros.org/wiki/xacro">
-    <xacro:include filename="modules/camlidarbot.xacro" />
+    <xacro:include filename="modules/chassis_and_wheels.xacro" />
+    <xacro:include filename="modules/camera.xacro" />
+    <xacro:include filename="modules/lidar.xacro" />
     <xacro:include filename="gazebo_tags/gazebo_plugins.xacro" />
     <xacro:include filename="gazebo_tags/gazebo_properties.xacro" />

Commit message: Modular xacro code improvements

File: urdf/gazebo_tags/gazebo_plugins.xacro (robot description, xacro)
@@ -11,7 +11,6 @@
             <wheel_separation>0.215</wheel_separation>
             <wheel_radius>0.06</wheel_radius>
-            <frame_id>camlidarbot/odom</frame_id> <!--Best to use prefixes ('camlidarbot' for example) and to set the prefix on the RVIZ config too-->
-            <child_frame_id>camlidarbot/base_footprint</child_frame_id> <!--Best to use prefixes ('camlidarbot' for example) and to set the prefix on the RVIZ config too-->
-            <!--<topic>cmd_vel</topic> -->
+            <frame_id>${robot_name}/odom</frame_id> <!--Best to use prefixes and to set the prefix on the RVIZ config too, see xacro_properties.xacro for where to change these -->
+            <child_frame_id>${robot_name}/base_footprint</child_frame_id>  <!--Best to use prefixes and to set the prefix on the RVIZ config too, see xacro_properties.xacro for where to change these -->
         </plugin>
     </gazebo>

File: urdf/modules/camera.xacro (robot description, xacro)
@@ -14,5 +14,5 @@
       <origin xyz="0 0 0" rpy="0 -0 0"/>
       <geometry>
-        <mesh filename="package://camlidarbot_description/assets/camera.stl"/>
+        <mesh filename="package://${package_name}/assets/camera.stl"/>
       </geometry>
       <material name="camera_material">
@@ -23,5 +23,5 @@
       <origin xyz="0 0 0" rpy="0 -0 0"/>
       <geometry>
-        <mesh filename="package://camlidarbot_description/assets/camera.stl"/>
+        <mesh filename="package://${package_name}/assets/camera.stl"/>
       </geometry>
     </collision>

File: urdf/modules/chassis_and_wheels.xacro (robot description, xacro)
@@ -22,5 +22,5 @@
       <origin xyz="0 0 0" rpy="0 -0 0"/>
       <geometry>
-        <mesh filename="package://camlidarbot_description/assets/chassis.stl"/>
+        <mesh filename="package://${package_name}/assets/chassis.stl"/>
       </geometry>
       <material name="chassis_material">
@@ -31,5 +31,5 @@
       <origin xyz="0 0 0" rpy="0 -0 0"/>
       <geometry>
-        <mesh filename="package://camlidarbot_description/assets/chassis.stl"/>
+        <mesh filename="package://${package_name}/assets/chassis.stl"/>
       </geometry>
     </collision>
@@ -46,5 +46,5 @@
       <origin xyz="0 0 0.0225" rpy="-1.5708 -0 0"/>
       <geometry>
-        <mesh filename="package://camlidarbot_description/assets/wheel.stl"/>
+        <mesh filename="package://${package_name}/assets/wheel.stl"/>
       </geometry>
       <material name="wheel_material">
@@ -55,5 +55,5 @@
       <origin xyz="0 0 0.0225" rpy="-1.5708 -0 0"/>
       <geometry>
-        <mesh filename="package://camlidarbot_description/assets/wheel.stl"/>
+        <mesh filename="package://${package_name}/assets/wheel.stl"/>
       </geometry>
     </collision>
@@ -78,5 +78,5 @@
       <origin xyz="0 0 0.0225" rpy="-1.5708 -0 0"/>
       <geometry>
-        <mesh filename="package://camlidarbot_description/assets/wheel.stl"/>
+        <mesh filename="package://${package_name}/assets/wheel.stl"/>
       </geometry>
       <material name="wheel_2_material">
@@ -87,5 +87,5 @@
       <origin xyz="0 0 0.0225" rpy="-1.5708 -0 0"/>
       <geometry>
-        <mesh filename="package://camlidarbot_description/assets/wheel.stl"/>
+        <mesh filename="package://${package_name}/assets/wheel.stl"/>
       </geometry>
     </collision>
@@ -110,5 +110,5 @@
       <origin xyz="0 0 0.0225" rpy="-1.5708 -0 0"/>
       <geometry>
-        <mesh filename="package://camlidarbot_description/assets/wheel.stl"/>
+        <mesh filename="package://${package_name}/assets/wheel.stl"/>
       </geometry>
       <material name="wheel_3_material">
@@ -119,5 +119,5 @@
       <origin xyz="0 0 0.0225" rpy="-1.5708 -0 0"/>
       <geometry>
-        <mesh filename="package://camlidarbot_description/assets/wheel.stl"/>
+        <mesh filename="package://${package_name}/assets/wheel.stl"/>
       </geometry>
     </collision>
@@ -142,5 +142,5 @@
       <origin xyz="0 0 0.0225" rpy="-1.5708 -0 0"/>
       <geometry>
-        <mesh filename="package://camlidarbot_description/assets/wheel.stl"/>
+        <mesh filename="package://${package_name}/assets/wheel.stl"/>
       </geometry>
       <material name="wheel_4_material">
@@ -151,5 +151,5 @@
       <origin xyz="0 0 0.0225" rpy="-1.5708 -0 0"/>
       <geometry>
-        <mesh filename="package://camlidarbot_description/assets/wheel.stl"/>
+        <mesh filename="package://${package_name}/assets/wheel.stl"/>
       </geometry>
     </collision>

File: urdf/modules/lidar.xacro (robot description, xacro)
@@ -14,5 +14,5 @@
       <origin xyz="0 -1.53081e-19 0" rpy="0 -0 0"/>
       <geometry>
-        <mesh filename="package://camlidarbot_description/assets/lidar.stl"/>
+        <mesh filename="package://${package_name}/assets/lidar.stl"/>
       </geometry>
       <material name="lidar_material">
@@ -23,5 +23,5 @@
       <origin xyz="0 -1.53081e-19 0" rpy="0 -0 0"/>
       <geometry>
-        <mesh filename="package://camlidarbot_description/assets/lidar.stl"/>
+        <mesh filename="package://${package_name}/assets/lidar.stl"/>
       </geometry>
     </collision>

File: urdf/robot.urdf.xacro (robot description, xacro)
@@ -1,4 +1,5 @@
 <?xml version="1.0" ?>
 <robot name="camlidarbot" xmlns:xacro="http://www.ros.org/wiki/xacro">
+    <xacro:include filename="xacro_properties/xacro_properties.xacro" />
     <xacro:include filename="modules/chassis_and_wheels.xacro" />
     <xacro:include filename="modules/camera.xacro" />
